File: pid_regulator.kicad_sch (KiCad schematic)
At the start: 12 parts, among them M1 Motor_DC, Q1 2N2222A, SW1 RotaryEncoder_Switch, U2 YD-ESP32-S3

Commit message: Add some minor changes
Signed-off-by: Volodymyr Kaliuzhnyi <vladimirvk2007@gmail.com>
Parts:
- renumbered C2 to C1, C1 to C2, R3 to R1, R4 to R2, R1 to R3, R2 to R4
Other:
- moved on the sheet: R1, R2
Changed lines of the file:
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@@
 	)
 	(junction
-		(at 179.07 113.03)
+		(at 142.24 113.03)
 		(diameter 0)
 		(color 0 0 0 0)
@@
 	)
 	(junction
-		(at 172.72 110.49)
+		(at 165.1 101.6)
+		(diameter 0)
+		(color 0 0 0 0)
+	)
+	(junction
+		(at 135.89 110.49)
 		(diameter 0)
 		(color 0 0 0 0)
@@
 	)
 	(junction
-		(at 172.72 100.33)
+		(at 135.89 100.33)
 		(diameter 0)
 		(color 0 0 0 0)
@@
 	(wire
 		(pts
-			(xy 172.72 110.49) (xy 184.15 110.49)
-		)
-		(stroke
-			(width 0)
-			(type default)
-		)
-	)
-	(wire
-		(pts
-			(xy 172.72 107.95) (xy 172.72 110.49)
+			(xy 135.89 110.49) (xy 184.15 110.49)
+		)
+		(stroke
+			(width 0)
+			(type default)
+		)
+	)
+	(wire
+		(pts
+			(xy 135.89 107.95) (xy 135.89 110.49)
 		)
 		(stroke
@@
 	(wire
 		(pts
-			(xy 172.72 99.06) (xy 172.72 100.33)
+			(xy 135.89 99.06) (xy 135.89 100.33)
 		)
 		(stroke
@@
 	(wire
 		(pts
-			(xy 179.07 107.95) (xy 179.07 113.03)
+			(xy 142.24 107.95) (xy 142.24 113.03)
 		)
 		(stroke
@@
 	(wire
 		(pts
-			(xy 127 110.49) (xy 172.72 110.49)
+			(xy 127 110.49) (xy 135.89 110.49)
 		)
 		(stroke
@@
 	(wire
 		(pts
-			(xy 127 113.03) (xy 179.07 113.03)
+			(xy 127 113.03) (xy 142.24 113.03)
+		)
+		(stroke
+			(width 0)
+			(type default)
+		)
+	)
+	(wire
+		(pts
+			(xy 165.1 101.6) (xy 165.1 104.14)
 		)
 		(stroke
@@
 	(wire
 		(pts
+			(xy 156.21 101.6) (xy 165.1 101.6)
+		)
+		(stroke
+			(width 0)
+			(type default)
+		)
+	)
+	(wire
+		(pts
 			(xy 198.12 105.41) (xy 198.12 104.14)
 		)
@@
 	(wire
 		(pts
-			(xy 179.07 113.03) (xy 189.23 113.03)
+			(xy 142.24 113.03) (xy 189.23 113.03)
 		)
 		(stroke
@@
 	(wire
 		(pts
-			(xy 172.72 100.33) (xy 179.07 100.33)
+			(xy 135.89 100.33) (xy 142.24 100.33)
 		)
 		(stroke
@@
 	(symbol
 		(lib_id "Device:R")
-		(at 179.07 104.14 180)
+		(at 142.24 104.14 180)
 		(unit 1)
 		(body_style 1)
@@
 		(in_pos_files yes)
 		(dnp no)
-		(property "Reference" "R4"
-			(at 180.34 104.14 0)
+		(property "Reference" "R2"
+			(at 143.51 104.14 0)
 			(show_name no)
 			(do_not_autoplace no)
@@
 		)
 		(property "Value" "4.7k"
-			(at 180.34 106.68 0)
+			(at 143.51 106.68 0)
 			(show_name no)
 			(do_not_autoplace no)
@@
 		)
 		(property "Footprint" ""
-			(at 180.848 104.14 90)
+			(at 144.018 104.14 90)
 			(hide yes)
 			(show_name no)
@@
 		)
 		(property "Datasheet" ""
-			(at 179.07 104.14 0)
+			(at 142.24 104.14 0)
 			(hide yes)
 			(show_name no)
@@
 		)
 		(property "Description" "Resistor"
-			(at 179.07 104.14 0)
+			(at 142.24 104.14 0)
 			(hide yes)
 			(show_name no)
@@
 			(project "pid_regulator"
 				(path "/7b671b88-447b-4e0a-a098-44d7aaa5c31d"
-					(reference "R4")
+					(reference "R2")
 					(unit 1)
 				)
@@
 		(dnp no)
 		(fields_autoplaced yes)
-		(property "Reference" "C1"
+		(property "Reference" "C2"
 			(at 212.09 107.0609 0)
 			(show_name no)
@@
 			(project "pid_regulator"
 				(path "/7b671b88-447b-4e0a-a098-44d7aaa5c31d"
-					(reference "C1")
+					(reference "C2")
 					(unit 1)
 				)
@@
 		(in_pos_files yes)
 		(dnp no)
-		(property "Reference" "R1"
+		(property "Reference" "R3"
 			(at 149.86 87.63 90)
 			(show_name no)
@@
 			(project "pid_regulator"
 				(path "/7b671b88-447b-4e0a-a098-44d7aaa5c31d"
-					(reference "R1")
+					(reference "R3")
 					(unit 1)
 				)
@@
 	(symbol
 		(lib_id "Device:R")
-		(at 172.72 104.14 180)
+		(at 135.89 104.14 180)
 		(unit 1)
 		(body_style 1)
@@
 		(in_pos_files yes)
 		(dnp no)
-		(property "Reference" "R3"
-			(at 173.99 104.14 0)
+		(property "Reference" "R1"
+			(at 137.16 104.14 0)
 			(show_name no)
 			(do_not_autoplace no)
@@
 		)
 		(property "Value" "4.7k"
-			(at 173.99 106.68 0)
+			(at 137.16 106.68 0)
 			(show_name no)
 			(do_not_autoplace no)
@@
 		)
 		(property "Footprint" ""
-			(at 174.498 104.14 90)
+			(at 137.668 104.14 90)
 			(hide yes)
 			(show_name no)
@@
 		)
 		(property "Datasheet" ""
-			(at 172.72 104.14 0)
+			(at 135.89 104.14 0)
 			(hide yes)
 			(show_name no)
@@
 		)
 		(property "Description" "Resistor"
-			(at 172.72 104.14 0)
+			(at 135.89 104.14 0)
 			(hide yes)
 			(show_name no)
@@
 			(project "pid_regulator"
 				(path "/7b671b88-447b-4e0a-a098-44d7aaa5c31d"
-					(reference "R3")
+					(reference "R1")
 					(unit 1)
 				)
@@
 	(symbol
 		(lib_id "power:+3.3V")
-		(at 172.72 99.06 0)
+		(at 135.89 99.06 0)
 		(unit 1)
 		(body_style 1)
@@
 		(fields_autoplaced yes)
 		(property "Reference" "#PWR010"
-			(at 172.72 102.87 0)
+			(at 135.89 102.87 0)
 			(hide yes)
 			(show_name no)
@@
 		)
 		(property "Value" "+3.3V"
-			(at 172.72 93.98 0)
+			(at 135.89 93.98 0)
 			(show_name no)
 			(do_not_autoplace no)
@@
 		)
 		(property "Footprint" ""
-			(at 172.72 99.06 0)
+			(at 135.89 99.06 0)
 			(hide yes)
 			(show_name no)
@@
 		)
 		(property "Datasheet" ""
-			(at 172.72 99.06 0)
+			(at 135.89 99.06 0)
 			(hide yes)
 			(show_name no)
@@
 		)
 		(property "Description" "Power symbol creates a global label with name \"+3.3V\""
-			(at 172.72 99.06 0)
+			(at 135.89 99.06 0)
 			(hide yes)
 			(show_name no)
@@
 	)
 	(symbol
-		(lib_id "power:GND")
-		(at 156.21 101.6 0)
-		(unit 1)
-		(body_style 1)
-		(exclude_from_sim no)
-		(in_bom yes)
-		(on_board yes)
-		(in_pos_files yes)
-		(dnp no)
-		(fields_autoplaced yes)
-		(property "Reference" "#PWR04"
-			(at 156.21 107.95 0)
-			(hide yes)
-			(show_name no)
-			(do_not_autoplace no)
-			(effects
-				(font
-					(size 1.27 1.27)
-				)
-			)
-		)
-		(property "Value" "GND"
-			(at 156.21 106.68 0)
-			(show_name no)
-			(do_not_autoplace no)
-			(effects
-				(font
-					(size 1.27 1.27)
-				)
-			)
-		)
-		(property "Footprint" ""
-			(at 156.21 101.6 0)
-			(hide yes)
-			(show_name no)
-			(do_not_autoplace no)
-			(effects
-				(font
-					(size 1.27 1.27)
-				)
-			)
-		)
-		(property "Datasheet" ""
-			(at 156.21 101.6 0)
-			(hide yes)
-			(show_name no)
-			(do_not_autoplace no)
-			(effects
-				(font
-					(size 1.27 1.27)
-				)
-			)
-		)
-		(property "Description" "Power symbol creates a global label with name \"GND\" , ground"
-			(at 156.21 101.6 0)
-			(hide yes)
-			(show_name no)
-			(do_not_autoplace no)
-			(effects
-				(font
-					(size 1.27 1.27)
-				)
-			)
-		)
-		(pin "1"
-		)
-		(instances
-			(project "pid_regulator"
-				(path "/7b671b88-447b-4e0a-a098-44d7aaa5c31d"
-					(reference "#PWR04")
-					(unit 1)
-				)
-			)
-		)
-	)
-	(symbol
 		(lib_id "Device:C")
 		(at 198.12 109.22 0)
@@
 		(in_pos_files yes)
 		(dnp no)
-		(property "Reference" "C2"
+		(property "Reference" "C1"
 			(at 200.66 106.68 0)
 			(show_name no)
@@
 			(project "pid_regulator"
 				(path "/7b671b88-447b-4e0a-a098-44d7aaa5c31d"
-					(reference "C2")
+					(reference "C1")
 					(unit 1)
 				)
@@
 	)
 	(symbol
-		(lib_id "power:GND")
-		(at 165.1 101.6 0)
+		(lib_id "power:GNDD")
+		(at 165.1 104.14 0)
 		(unit 1)
 		(body_style 1)
@@
 		(dnp no)
 		(fields_autoplaced yes)
-		(property "Reference" "#PWR02"
+		(property "Reference" "#PWR024"
+			(at 165.1 110.49 0)
+			(hide yes)
+			(show_name no)
+			(do_not_autoplace no)
+			(effects
+				(font
+					(size 1.27 1.27)
+				)
+			)
+		)
+		(property "Value" "GNDD"
 			(at 165.1 107.95 0)
-			(hide yes)
-			(show_name no)
-			(do_not_autoplace no)
-			(effects
-				(font
-					(size 1.27 1.27)
-				)
-			)
-		)
-		(property "Value" "GND"
-			(at 165.1 106.68 0)
 			(show_name no)
 			(do_not_autoplace no)
@@
 		)
 		(property "Footprint" ""
-			(at 165.1 101.6 0)
+			(at 165.1 104.14 0)
 			(hide yes)
 			(show_name no)
@@
 		)
 		(property "Datasheet" ""
-			(at 165.1 101.6 0)
-			(hide yes)
-			(show_name no)
-			(do_not_autoplace no)
-			(effects
-				(font
-					(size 1.27 1.27)
-				)
-			)
-		)
-		(property "Description" "Power symbol creates a global label with name \"GND\" , ground"
-			(at 165.1 101.6 0)
+			(at 165.1 104.14 0)
+			(hide yes)
+			(show_name no)
+			(do_not_autoplace no)
+			(effects
+				(font
+					(size 1.27 1.27)
+				)
+			)
+		)
+		(property "Description" "Power symbol creates a global label with name \"GNDD\" , digital ground"
+			(at 165.1 104.14 0)
 			(hide yes)
 			(show_name no)
@@
 			(project "pid_regulator"
 				(path "/7b671b88-447b-4e0a-a098-44d7aaa5c31d"
-					(reference "#PWR02")
+					(reference "#PWR024")
 					(unit 1)
 				)
@@
 		(in_pos_files yes)
 		(dnp no)
-		(property "Reference" "R2"
+		(property "Reference" "R4"
 			(at 157.48 96.52 0)
 			(show_name no)
@@
 			(project "pid_regulator"
 				(path "/7b671b88-447b-4e0a-a098-44d7aaa5c31d"
-					(reference "R2")
+					(reference "R4")
 					(unit 1)
 				)
